File: Camera-Wing-SHIM/Camera-Wing-SHIM.kicad_sch (KiCad schematic)
At the start: 2 parts, among them J1 Pico RHS Headers, J2 Pin Connection

Commit message: Fixed
Parts:
- added J3: Pin Connection, Connector_PinHeader_2.54mm:PinHeader_1x06_P2.54mm_Vertical, symbol Connector:Conn_01x06_Pin
- J2: value Pin Connection -> SMD Header Connection
Connections:
- net +3V3: now also J1.5 (Pin_5), J3.1 (Pin_1); no longer J1.3 (Pin_3)
- net CLK: now also J3.3 (Pin_3)
- net CS: now also J3.6 (Pin_6)
- net GND: now also J1.3 (Pin_3), J3.2 (Pin_2); no longer J1.5 (Pin_5)
- net MISO: now also J3.4 (Pin_4)
- net MOSI: now also J3.5 (Pin_5)
Changed lines of the file:
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@@
+    (stroke (width 0) (type default))
+  )
+  (wire (pts (xy 71.12 59.69) (xy 86.36 59.69))
+    (stroke (width 0) (type default))
+  )
+  (wire (pts (xy 133.35 73.66) (xy 139.7 73.66))
+    (stroke (width 0) (type default))
+  )
+  (wire (pts (xy 147.32 68.58) (xy 147.32 66.04))
+    (stroke (width 0) (type default))
+  )
+  (wire (pts (xy 167.64 81.28) (xy 173.99 81.28))
+    (stroke (width 0) (type default))
+  )
+  (wire (pts (xy 133.35 71.12) (xy 147.32 71.12))
+    (stroke (width 0) (type default))
+  )
+  (wire (pts (xy 167.64 76.2) (xy 173.99 76.2))
+    (stroke (width 0) (type default))
+  )
+  (wire (pts (xy 80.01 54.61) (xy 80.01 55.88))
+    (stroke (width 0) (type default))
+  )
+  (wire (pts (xy 167.64 73.66) (xy 173.99 73.66))
+    (stroke (width 0) (type default))
+  )
+  (wire (pts (xy 167.64 71.12) (xy 181.61 71.12))
+    (stroke (width 0) (type default))
+  )
+  (wire (pts (xy 167.64 78.74) (xy 173.99 78.74))
+    (stroke (width 0) (type default))
+  )
+  (wire (pts (xy 71.12 92.71) (xy 92.71 92.71))
+    (stroke (width 0) (type default))
+  )
+  (wire (pts (xy 92.71 92.71) (xy 92.71 95.25))
+    (stroke (width 0) (type default))
+  )
+  (wire (pts (xy 181.61 68.58) (xy 181.61 66.04))
+    (stroke (width 0) (type default))
+  )
+  (wire (pts (xy 71.12 90.17) (xy 82.55 90.17))
+    (stroke (width 0) (type default))
+  )
+  (wire (pts (xy 71.12 87.63) (xy 82.55 87.63))
+    (stroke (width 0) (type default))
+  )
+  (wire (pts (xy 86.36 59.69) (xy 86.36 57.15))
+    (stroke (width 0) (type default))
+  )
+  (wire (pts (xy 147.32 71.12) (xy 147.32 73.66))
+    (stroke (width 0) (type default))
+  )
+  (wire (pts (xy 167.64 68.58) (xy 181.61 68.58))
+    (stroke (width 0) (type default))
+  )
+  (wire (pts (xy 133.35 76.2) (xy 139.7 76.2))
+    (stroke (width 0) (type default))
+  )
+  (wire (pts (xy 71.12 97.79) (xy 82.55 97.79))
     (stroke (width 0) (type default))
   )
@@
     (stroke (width 0) (type default))
   )
-  (wire (pts (xy 133.35 73.66) (xy 139.7 73.66))
-    (stroke (width 0) (type default))
-  )
-  (wire (pts (xy 147.32 68.58) (xy 147.32 66.04))
-    (stroke (width 0) (type default))
-  )
-  (wire (pts (xy 133.35 71.12) (xy 147.32 71.12))
-    (stroke (width 0) (type default))
-  )
-  (wire (pts (xy 80.01 59.69) (xy 80.01 62.23))
-    (stroke (width 0) (type default))
-  )
-  (wire (pts (xy 71.12 92.71) (xy 92.71 92.71))
-    (stroke (width 0) (type default))
-  )
-  (wire (pts (xy 92.71 92.71) (xy 92.71 95.25))
-    (stroke (width 0) (type default))
-  )
-  (wire (pts (xy 71.12 90.17) (xy 82.55 90.17))
-    (stroke (width 0) (type default))
-  )
-  (wire (pts (xy 71.12 87.63) (xy 82.55 87.63))
-    (stroke (width 0) (type default))
-  )
-  (wire (pts (xy 80.01 54.61) (xy 80.01 52.07))
-    (stroke (width 0) (type default))
-  )
-  (wire (pts (xy 147.32 71.12) (xy 147.32 73.66))
-    (stroke (width 0) (type default))
-  )
-  (wire (pts (xy 133.35 76.2) (xy 139.7 76.2))
-    (stroke (width 0) (type default))
-  )
-  (wire (pts (xy 71.12 97.79) (xy 82.55 97.79))
-    (stroke (width 0) (type default))
-  )
-  (wire (pts (xy 71.12 59.69) (xy 80.01 59.69))
-    (stroke (width 0) (type default))
-  )
   (wire (pts (xy 133.35 81.28) (xy 139.7 81.28))
     (stroke (width 0) (type default))
   )
+  (wire (pts (xy 181.61 71.12) (xy 181.61 73.66))
+    (stroke (width 0) (type default))
+  )
   (wire (pts (xy 133.35 68.58) (xy 147.32 68.58))
     (stroke (width 0) (type default))
@@
     (effects (font (size 1.27 1.27)) (justify right bottom))
   )
+  (label "CS" (at 173.99 81.28 180) (fields_autoplaced)
+    (effects (font (size 1.27 1.27)) (justify right bottom))
+  )
+  (label "MISO" (at 173.99 76.2 180) (fields_autoplaced)
+    (effects (font (size 1.27 1.27)) (justify right bottom))
+  )
   (label "MISO" (at 82.55 97.79 180) (fields_autoplaced)
     (effects (font (size 1.27 1.27)) (justify right bottom))
@@
     (effects (font (size 1.27 1.27)) (justify right bottom))
   )
+  (label "MOSI" (at 173.99 78.74 180) (fields_autoplaced)
+    (effects (font (size 1.27 1.27)) (justify right bottom))
+  )
+  (label "CLK" (at 173.99 73.66 180) (fields_autoplaced)
+    (effects (font (size 1.27 1.27)) (justify right bottom))
+  )
   (label "CS" (at 139.7 81.28 180) (fields_autoplaced)
     (effects (font (size 1.27 1.27)) (justify right bottom))
@@
     (effects (font (size 1.27 1.27)) (justify right bottom))
   )
-  (symbol (lib_id "power:GND") (at 80.01 62.23 0) (unit 1)
-    (in_bom yes) (on_board yes) (dnp no) (fields_autoplaced)
-    (property "Reference" "#PWR02" (at 80.01 68.58 0)
-      (effects (font (size 1.27 1.27)) hide)
-    )
-    (property "Value" "GND" (at 80.01 67.31 0)
-      (effects (font (size 1.27 1.27)))
-    )
-    (property "Footprint" "" (at 80.01 62.23 0)
-      (effects (font (size 1.27 1.27)) hide)
-    )
-    (property "Datasheet" "" (at 80.01 62.23 0)
+  (symbol (lib_id "power:GND") (at 80.01 55.88 0) (unit 1)
+    (in_bom yes) (on_board yes) (dnp no)
+    (property "Reference" "#PWR02" (at 80.01 62.23 0)
+      (effects (font (size 1.27 1.27)) hide)
+    )
+    (property "Value" "GND" (at 80.01 53.34 0)
+      (effects (font (size 1.27 1.27)))
+    )
+    (property "Footprint" "" (at 80.01 55.88 0)
+      (effects (font (size 1.27 1.27)) hide)
+    )
+    (property "Datasheet" "" (at 80.01 55.88 0)
       (effects (font (size 1.27 1.27)) hide)
     )
@@
       (effects (font (size 1.27 1.27)))
     )
-    (property "Value" "Pin Connection" (at 128.905 66.04 0)
+    (property "Value" "SMD Header Connection" (at 128.905 66.04 0)
       (effects (font (size 1.27 1.27)))
     )
@@
     )
   )
+  (symbol (lib_id "Connector:Conn_01x06_Pin") (at 162.56 73.66 0) (unit 1)
+    (in_bom yes) (on_board yes) (dnp no) (fields_autoplaced)
+    (property "Reference" "J3" (at 163.195 63.5 0)
+      (effects (font (size 1.27 1.27)))
+    )
+    (property "Value" "Pin Connection" (at 163.195 66.04 0)
+      (effects (font (size 1.27 1.27)))
+    )
+    (property "Footprint" "Connector_PinHeader_2.54mm:PinHeader_1x06_P2.54mm_Vertical" (at 162.56 73.66 0)
+      (effects (font (size 1.27 1.27)) hide)
+    )
+    (property "Datasheet" "~" (at 162.56 73.66 0)
+      (effects (font (size 1.27 1.27)) hide)
+    )
+    (pin "6")
+    (pin "4")
+    (pin "3")
+    (pin "1")
+    (pin "5")
+    (pin "2")
+    (instances
+      (project "Camera-Wing-SHIM"
+        (path "/573a4d9c-bd0f-4c16-a1f5-7ab3d68c8cde"
+          (reference "J3") (unit 1)
+        )
+      )
+    )
+  )
   (symbol (lib_id "power:GND") (at 92.71 95.25 0) (unit 1)
     (in_bom yes) (on_board yes) (dnp no) (fields_autoplaced)
@@
     )
   )
-  (symbol (lib_id "power:+3V3") (at 80.01 52.07 0) (unit 1)
-    (in_bom yes) (on_board yes) (dnp no) (fields_autoplaced)
-    (property "Reference" "#PWR01" (at 80.01 55.88 0)
-      (effects (font (size 1.27 1.27)) hide)
-    )
-    (property "Value" "+3V3" (at 80.01 46.99 0)
-      (effects (font (size 1.27 1.27)))
-    )
-    (property "Footprint" "" (at 80.01 52.07 0)
-      (effects (font (size 1.27 1.27)) hide)
-    )
-    (property "Datasheet" "" (at 80.01 52.07 0)
-      (effects (font (size 1.27 1.27)) hide)
-    )
+  (symbol (lib_id "power:+3V3") (at 181.61 66.04 0) (unit 1)
+    (in_bom yes) (on_board yes) (dnp no) (fields_autoplaced)
+    (property "Reference" "#PWR06" (at 181.61 69.85 0)
+      (effects (font (size 1.27 1.27)) hide)
+    )
+    (property "Value" "+3V3" (at 181.61 60.96 0)
+      (effects (font (size 1.27 1.27)))
+    )
+    (property "Footprint" "" (at 181.61 66.04 0)
+      (effects (font (size 1.27 1.27)) hide)
+    )
+    (property "Datasheet" "" (at 181.61 66.04 0)
+      (effects (font (size 1.27 1.27)) hide)
+    )
+    (pin "1")
+    (instances
+      (project "Camera-Wing-SHIM"
+        (path "/573a4d9c-bd0f-4c16-a1f5-7ab3d68c8cde"
+          (reference "#PWR06") (unit 1)
+        )
+      )
+    )
+  )
+  (symbol (lib_id "power:GND") (at 181.61 73.66 0) (unit 1)
+    (in_bom yes) (on_board yes) (dnp no) (fields_autoplaced)
+    (property "Reference" "#PWR07" (at 181.61 80.01 0)
+      (effects (font (size 1.27 1.27)) hide)
+    )
+    (property "Value" "GND" (at 181.61 78.74 0)
+      (effects (font (size 1.27 1.27)))
+    )
+    (property "Footprint" "" (at 181.61 73.66 0)
+      (effects (font (size 1.27 1.27)) hide)
+    )
+    (property "Datasheet" "" (at 181.61 73.66 0)
+      (effects (font (size 1.27 1.27)) hide)
+    )
+    (pin "1")
+    (instances
+      (project "Camera-Wing-SHIM"
+        (path "/573a4d9c-bd0f-4c16-a1f5-7ab3d68c8cde"
+          (reference "#PWR07") (unit 1)
+        )
+      )
+    )
+  )
+  (symbol (lib_id "power:+3V3") (at 86.36 57.15 0) (unit 1)
+    (in_bom yes) (on_board yes) (dnp no)
+    (property "Reference" "#PWR01" (at 86.36 60.96 0)
+      (effects (font (size 1.27 1.27)) hide)
+    )
+    (property "Value" "+3V3" (at 86.36 53.34 0)
+      (effects (font (size 1.27 1.27)))
+    )
+    (property "Footprint" "" (at 86.36 57.15 0)
+      (effects (font (size 1.27 1.27)) hide)
+    )
+    (property "Datasheet" "" (at 86.36 57.15 0)
+      (effects (font (size 1.27 1.27)) hide)
+    )
